File: Electronics/RFControllerKiCAD/RFController.kicad_pcb (KiCad board)
At the start: 2 copper layers, 191.5 x 193.3 mm, 17 parts, among them SW1 SW_Push, SW2 SW_Push, SW3 SW_Push, SW4 SW_Push, SW5 SW_Push, SW6 SW_Push

Commit message: Updated STLs
Parts:
- moved Radio1 44.9 mm to (168.1, 70.1)
- moved C1 36.5 mm to (156.5, 97.0), turned to 180 degrees
- renumbered G*** to C-3P0, G*** to R2-D2
Routing:
- net +3.3V: track 152.2 -> 219.7 mm
- net /MOSI: track 34.2 -> 80.3 mm
- net /SCK: track 19.4 -> 64.5 mm
- net /CE: track 20.9 -> 65.5 mm
- net /MISO: track 26.2 -> 67.7 mm
- net /CSN: track 42.8 -> 77.1 mm
- net GND: vias 2945 -> 2872
Other:
- outline, holes or cut-outs redrawn
